Commit message: sim

File: wpr1_bringup/urdf/wpr1.urdf (robot description, URDF)
Before this commit: robot WPR1, 17 links, 16 joints
Joints:
- joint base_joint1: origin xyz=0.185 0.05 0.515 rpy=0 1.57 0 -> xyz=0.185 0.00 0.515 rpy=0 1.57 0

File: wpr1_bringup/urdf/wpr1_moveit.urdf (robot description, URDF)
Before this commit: robot WPR1, 17 links, 16 joints
Links:
- added link dummy
Joints:
- added joint dummy_joint: type fixed, parent dummy, child base_footprint
- joint base_joint1: origin xyz=0.185 0.05 0.515 rpy=0 1.57 0 -> xyz=0.185 0.00 0.515 rpy=0 1.57 0
