Commit message: grab value

File: wpr1_bringup/urdf/wpr1_moveit.urdf (robot description, URDF)
Before this commit: robot WPR1, 18 links, 17 joints
Links:
- removed link dummy
Joints:
- removed joint dummy_joint
- joint base_joint1: origin xyz=0.185 0.00 0.515 rpy=0 1.57 0 -> xyz=0.185 0.05 0.515 rpy=0 1.57 0

Commit message: urdf for moveit

File: wpr1_bringup/urdf/wpr1_moveit.urdf (robot description, URDF)
Before this commit: robot WPR1, 17 links, 16 joints
Joints:
- joint base_joint1: origin xyz=0.185 0.05 0.515 rpy=0 1.57 0 -> xyz=0.185 0.00 0.515 rpy=0 1.57 0

Commit message: new urdf_moveit

File: wpr1_bringup/urdf/wpr1_moveit.urdf (robot description, URDF)
Before this commit: robot WPR1, 17 links, 16 joints
Joints:
- joint 0_torso_lift: axis 0 0 1 -> 1 0 0; origin xyz=-0.255 0 0.287 rpy=0 0 0 -> xyz=-0.255 0 0.287 rpy=0 -1.57 0
- joint 1_shoulder_roll: axis 0 0 1 -> 1 0 0; origin xyz=0 0 0.1585 -> xyz=0.1585 0 0
- joint 2_shoulder_flex: origin xyz=0 0 0.0825 -> xyz=0.0825 0 0
- joint 3_upperarm_roll: axis 0 0 1 -> 1 0 0; origin xyz=0 0 0.197 -> xyz=0.197 0 0
- joint 4_elbow_flex: axis 1 0 0 -> 0 0 -1; origin xyz=0 0 0.076 -> xyz=0.076 0 0
- joint 5_forearm_roll: axis 0 0 1 -> 1 0 0; origin xyz=0 0 0.197 -> xyz=0.197 0 0
- joint 6_wrist_flex: origin xyz=0 0 0.076 -> xyz=0.076 0 0
- joint 7_gripper: axis -1 0 0 -> 0 0 1; origin xyz=0 0.06 0.219 -> xyz=0.219 0.06 0
- joint base_joint1: origin xyz=0.185 0.00 0.515 rpy=0 1.57 0 -> xyz=0.515 0.00 -0.185 rpy=0 1.57 0
- joint kinect_height: origin xyz=0.174 0 0 rpy=0 -1.5707963 0 -> xyz=0 0 -0.174 rpy=0 0 0
- joint palm_tip: origin xyz=0 0 0.32 rpy=0 -1.57 0 -> xyz=0.32 0 0 rpy=0 0 0
- joint wpm2_palm_right_finger: axis 1 0 0 -> 0 0 -1; origin xyz=0 -0.06 0.219 -> xyz=0.219 -0.06 0
